Commit message: basic slam with phobos_nuclear now working

File: i3dr_tools_ros_WS/src/i3dr_cameras/i3dr_phobos_nuclear-ros/urdf/phobos_nuclear_scene.urdf.xacro (robot description, xacro)
@@ -6,4 +6,4 @@
     xmlns:xacro="http://ros.org/wiki/xacro">
     <xacro:include filename="$(find i3dr_stereo_camera)/urdf/i3dr_stereo_camera.urdf.xacro" />
-    <xacro:i3dr_stereo_camera camera_name="phobos_nuclear" baseline="0.25" toe_in="0" width="0.038" height="0.10175" length="0.03242" mount_offset_y="-0.015" image_width="1920" image_height="1080" image_format="MONO8" hfov="1.04" focus_near="0.3" r="0.1" g="0.1" b="0.1" />
+    <xacro:i3dr_stereo_camera camera_name="phobos_nuclear" baseline="0.25" toe_in_r="7" toe_in_l="0" width="0.05" height="0.3" length="0.05" image_width="1920" image_height="1080" image_format="MONO8" hfov="1.04" focus_near="0.3" r="0.1" g="0.1" b="0.1" />
 </robot>

File: i3dr_tools_ros_WS/src/i3dr_cameras/i3dr_stereo_camera-ros/urdf/example_camera.urdf.xacro (robot description, xacro)
@@ -6,4 +6,4 @@
     xmlns:xacro="http://ros.org/wiki/xacro">
     <xacro:include filename="$(find i3dr_custom_camera-ros)/urdf/i3dr_stereo_camera.urdf.xacro" />
-    <xacro:i3dr_stereo_camera camera_name="example_camera" baseline="0.06" toe_in="0" width="0.038" height="0.10175" length="0.03242" mount_offset_y="-0.015" image_width="752" image_height="480" image_format="MONO8" hfov="1.04" focus_near="0.3" r="0.1" g="0.1" b="0.1" />
+    <xacro:i3dr_stereo_camera camera_name="example_camera" baseline="0.06" toe_in_r="0" toe_in_l="0" width="0.038" height="0.10175" length="0.03242" mount_offset_y="-0.015" image_width="752" image_height="480" image_format="MONO8" hfov="1.04" focus_near="0.3" r="0.1" g="0.1" b="0.1" />
 </robot>

File: i3dr_tools_ros_WS/src/i3dr_cameras/i3dr_stereo_camera-ros/urdf/i3dr_stereo_camera.urdf.xacro (robot description, xacro)
@@ -4,5 +4,5 @@
 -->
 <robot xmlns:xacro="http://ros.org/wiki/xacro">
-    <xacro:macro name="i3dr_stereo_camera" params="camera_name baseline toe_in width height length image_format:=RGB8 image_height:=640 image_width:=480 hfov:=1.579 focus_near:=0 focus_far:=100 camera_offset_x:=0 camera_offset_y:=0 camera_offset_z:=0 mount_offset_x:=0 mount_offset_y:=0 mount_offset_z:=0 r:=1 g:=0 b:=0 a:=1">
+    <xacro:macro name="i3dr_stereo_camera" params="camera_name baseline toe_in_r toe_in_l width height length image_format:=RGB8 image_height:=640 image_width:=480 hfov:=1.579 focus_near:=0 focus_far:=100 camera_offset_x:=0 camera_offset_y:=0 camera_offset_z:=0 mount_offset_x:=0 mount_offset_y:=0 mount_offset_z:=0 r:=1 g:=0 b:=0 a:=1">
         <link name="${camera_name}_cameraLeft_optical" />
         <link name="${camera_name}_cameraRight_optical" />
@@ -36,5 +36,5 @@
             <child link="${camera_name}_cameraLeft_optical"/>
             <!-- Correct for the optical frame orientation -->
-            <origin xyz="0 0 0" rpy="${-pi/2} 0 ${(-pi/2)-toe_in}" />
+            <origin xyz="0 0 0" rpy="${-pi/2} 0 ${(-pi/2)-(toe_in_l * (pi/180))}" />
         </joint>
         <joint name="${camera_name}_right_optical_joint" type="fixed">
@@ -42,5 +42,5 @@
             <child link="${camera_name}_cameraRight_optical"/>
             <!-- Correct for the optical frame orientation -->
-            <origin xyz="0 0 0" rpy="${-pi/2} 0 ${(-pi/2)+toe_in}" />
+            <origin xyz="0 0 0" rpy="${-pi/2} 0 ${(-pi/2)+(toe_in_r * (pi/180))}" />
         </joint>
         <sensor name="${camera_name}_right_camera_sensor" update_rate="60">
