Commit message: Update to registration for phobos nuclear

File: i3dr_tools_ros_WS/src/i3dr_cameras/i3dr_phobos-ros/urdf/standalone.urdf.xacro (robot description, xacro)
@@ -1,5 +1,5 @@
 <?xml version="1.0"?>
 <robot name="phobos" xmlns:xacro="http://ros.org/wiki/xacro">
-  <xacro:include filename="$(find phobos)/urdf/phobos.urdf.xacro" />
+  <xacro:include filename="$(find i3dr_phobos)/urdf/phobos.urdf.xacro" />
   <link name="base_link" />
   <xacro:phobos_camera />

File: i3dr_tools_ros_WS/src/i3dr_cameras/i3dr_stereo_camera-ros/urdf/i3dr_stereo_camera.urdf.xacro (robot description, xacro)
@@ -60,5 +60,5 @@
             <parent link="${camera_name}_base_link"/>
             <child link="${camera_name}_center"/>
-            <origin xyz="${mount_offset_x} ${mount_offset_y} ${(length/2)+mount_offset_z}" rpy="0 0 0" />
+            <origin xyz="${mount_offset_x} ${mount_offset_y} ${(length/2)+mount_offset_z}" rpy="0 0 ${-pi/2}" />
         </joint>
         <!-- Correct for IMU orientation, Z -> X -->
