Commit message: improvements to rtabmap intergration with cameras

File: i3dr_tools_ros_WS/src/i3dr_cameras/i3dr_deimos-ros/urdf/deimos_scene.urdf.xacro (robot description, xacro)
@@ -6,4 +6,4 @@
     xmlns:xacro="http://ros.org/wiki/xacro">
     <xacro:include filename="$(find i3dr_stereo_camera)/urdf/i3dr_stereo_camera.urdf.xacro" />
-    <xacro:i3dr_stereo_camera camera_name="deimos" baseline="0.06" toe_in="0" width="0.038" height="0.10175" length="0.03242" mount_offset_y="-0.015" image_width="752" image_height="480" image_format="MONO8" hfov="1.04" focus_near="0.3" r="0.1" g="0.1" b="0.1" />
+    <xacro:i3dr_stereo_camera camera_name="deimos" baseline="0.06" toe_in_r="0" toe_in_l="0" width="0.038" height="0.10175" length="0.03242" mount_offset_y="-0.015" image_width="752" image_height="480" image_format="MONO8" hfov="1.04" focus_near="0.3" r="0.1" g="0.1" b="0.1" />
 </robot>

File: i3dr_tools_ros_WS/src/i3dr_cameras/i3dr_stereo_camera-ros/urdf/i3dr_stereo_camera.urdf.xacro (robot description, xacro)
@@ -9,4 +9,5 @@
         <link name="${camera_name}_cameraLeft" />
         <link name="${camera_name}_cameraRight" />
+        <link name="${camera_name}_depth_optical_frame" />
         <link name="${camera_name}_base_link" />
         <!--<link name="imu_link"/>-->
@@ -44,4 +45,9 @@
             <origin xyz="0 0 0" rpy="${-pi/2} 0 ${(-pi/2)+(toe_in_r * (pi/180))}" />
         </joint>
+        <joint name="${camera_name}_depth_optical_joint" type="fixed">
+            <parent link="${camera_name}_cameraLeft_optical"/>
+            <child link="${camera_name}_depth_optical_frame"/>
+            <origin xyz="0 0 0" rpy="0 0 0" />
+        </joint>
         <sensor name="${camera_name}_right_camera_sensor" update_rate="60">
             <parent link="${camera_name}_cameraRight_optical"/>

Commit message: add submodules

File: i3dr_tools_ros_WS/src/i3dr_cameras/i3dr_deimos-ros/urdf/deimos_scene.urdf.xacro (robot description, xacro)
@@ -5,5 +5,10 @@
 <robot name="deimos"
     xmlns:xacro="http://ros.org/wiki/xacro">
+    <!--<link name="odom"/>-->
     <xacro:include filename="$(find i3dr_stereo_camera)/urdf/i3dr_stereo_camera.urdf.xacro" />
     <xacro:i3dr_stereo_camera camera_name="deimos" baseline="0.06" toe_in_r="0" toe_in_l="0" width="0.038" height="0.10175" length="0.03242" mount_offset_y="-0.015" image_width="752" image_height="480" image_format="MONO8" hfov="1.04" focus_near="0.3" r="0.1" g="0.1" b="0.1" />
+    <!--<joint name="world_imu_joint" type="floating">
+        <parent link="deimos_imu_link"/>
+        <child link="odom"/>
+    </joint>-->
 </robot>

File: i3dr_tools_ros_WS/src/i3dr_cameras/i3dr_phobos-ros/urdf/phobos_scene.urdf.xacro (robot description, xacro)
@@ -6,4 +6,16 @@
     xmlns:xacro="http://ros.org/wiki/xacro">
     <xacro:include filename="$(find i3dr_stereo_camera)/urdf/i3dr_stereo_camera.urdf.xacro" />
-    <xacro:i3dr_stereo_camera camera_name="phobos" baseline="0.28" toe_in_r="8.5" toe_in_l="8.5" width="0.05" height="0.3" length="0.05" image_width="1920" image_height="1080" image_format="MONO8" hfov="1.04" focus_near="0.3" r="0.1" g="0.1" b="0.1" />
+    <xacro:i3dr_stereo_camera camera_name="phobos" baseline="0.28" toe_in_r="8.5" toe_in_l="8.5" width="0.05" height="0.3" length="0.05" image_width="1920" image_height="1080" image_format="MONO8" hfov="1.04" focus_near="0.3" r="1" g="0.5" b="0.1" />
+    <link name="aruco_marker_left"/>
+    <link name="aruco_marker_right"/>>
+    <joint name="arcuo_l_phobos_joint" type="fixed">
+        <parent link="phobos_cameraLeft_optical"/>
+        <child link="aruco_marker_left"/>
+        <origin xyz="0 0 0" rpy="0 0 0" />
+    </joint>
+    <joint name="arcuo_r_phobos_joint" type="fixed">
+        <parent link="phobos_cameraRight_optical"/>
+        <child link="aruco_marker_right"/>
+        <origin xyz="0 0 0" rpy="0 0 0" />
+    </joint>
 </robot>

File: i3dr_tools_ros_WS/src/i3dr_cameras/i3dr_stereo_camera-ros/urdf/i3dr_stereo_camera.urdf.xacro (robot description, xacro)
@@ -11,5 +11,5 @@
         <link name="${camera_name}_depth_optical_frame" />
         <link name="${camera_name}_base_link" />
-        <!--<link name="imu_link"/>-->
+        <link name="${camera_name}_imu_link"/>
         <link name="${camera_name}_center">
             <visual>
@@ -26,4 +26,5 @@
             <parent link="${camera_name}_center"/>
             <child link="${camera_name}_cameraRight"/>
+            <!--<origin xyz="0 -0.1447027  0" rpy="0 0 0"/>-->
             <origin xyz="${camera_offset_x} -${(baseline/2)+camera_offset_y} ${camera_offset_z}" rpy="0 0 0" />
         </joint>
@@ -31,4 +32,5 @@
             <parent link="${camera_name}_center"/>
             <child link="${camera_name}_cameraLeft"/>
+            <!--<origin xyz="0 0.1447027  0" rpy="0 0 0"/>-->
             <origin xyz="${camera_offset_x} ${(baseline/2)+camera_offset_y} ${camera_offset_z}" rpy="0 0 0" />
         </joint>
@@ -63,9 +65,9 @@
         </joint>
         <!-- Correct for IMU orientation, Z -> X -->
-        <!--<joint name="${camera_name}_imu_joint" type="fixed">
+        <joint name="${camera_name}_imu_joint" type="fixed">
             <origin xyz="0 0.015 -0.002" rpy="0 ${pi/2} 0" />
-            <parent link="${camera_name}_center" />
-            <child link="imu_link" />
-        </joint>-->
+            <parent link="${camera_name}_imu_link" />
+            <child link="${camera_name}_base_link" />
+        </joint>
     </xacro:macro>
 </robot>
