Commit message: Fix point cloud publishing using i3dr_point_cloud node

File: i3dr_tools_ros_WS/src/i3dr_cameras/i3dr_deimos-ros/urdf/deimos_scene.urdf.xacro (robot description, xacro)
@@ -7,5 +7,5 @@
     <!--<link name="odom"/>-->
     <xacro:include filename="$(find i3dr_stereo_camera)/urdf/i3dr_stereo_camera.urdf.xacro" />
-    <xacro:i3dr_stereo_camera camera_name="deimos" baseline="0.06" toe_in_r="0" toe_in_l="0" width="0.038" height="0.10175" length="0.03242" mount_offset_y="-0.015" image_width="752" image_height="480" image_format="MONO8" hfov="1.04" focus_near="0.3" r="0.1" g="0.1" b="0.1" />
+    <xacro:i3dr_stereo_camera camera_name="deimos" baseline="0.06" toe_in_r="0" toe_in_l="0" width="0.10175" height="0.038" length="0.03242" mount_offset_y="-0.015" image_width="752" image_height="480" image_format="MONO8" hfov="1.04" focus_near="0.3" r="0.1" g="0.1" b="0.1" />
     <!--<joint name="world_imu_joint" type="floating">
         <parent link="deimos_imu_link"/>

File: i3dr_tools_ros_WS/src/i3dr_cameras/i3dr_phobos-ros/urdf/phobos_scene.urdf.xacro (robot description, xacro)
@@ -6,5 +6,5 @@
     xmlns:xacro="http://ros.org/wiki/xacro">
     <xacro:include filename="$(find i3dr_stereo_camera)/urdf/i3dr_stereo_camera.urdf.xacro" />
-    <xacro:i3dr_stereo_camera camera_name="phobos" baseline="0.28" toe_in_r="8.5" toe_in_l="8.5" width="0.05" height="0.3" length="0.05" image_width="1920" image_height="1080" image_format="MONO8" hfov="1.04" focus_near="0.3" r="1" g="0.5" b="0.1" />
+    <xacro:i3dr_stereo_camera camera_name="phobos" baseline="0.28" toe_in_r="8.5" toe_in_l="8.5" width="0.39" height="0.05" length="0.14" image_width="1920" image_height="1080" image_format="MONO8" hfov="1.04" focus_near="0.3" r="1" g="0.5" b="0.1" />
     <link name="aruco_marker_left"/>
     <link name="aruco_marker_right"/>>

File: i3dr_tools_ros_WS/src/i3dr_cameras/i3dr_phobos_nuclear-ros/urdf/phobos_nuclear_scene.urdf.xacro (robot description, xacro)
@@ -6,4 +6,4 @@
     xmlns:xacro="http://ros.org/wiki/xacro">
     <xacro:include filename="$(find i3dr_stereo_camera)/urdf/i3dr_stereo_camera.urdf.xacro" />
-    <xacro:i3dr_stereo_camera camera_name="phobos_nuclear" baseline="0.25" toe_in_r="7" toe_in_l="0" width="0.05" height="0.3" length="0.05" image_width="1920" image_height="1080" image_format="MONO8" hfov="1.04" focus_near="0.3" r="0.1" g="0.1" b="0.1" />
+    <xacro:i3dr_stereo_camera camera_name="phobos_nuclear" baseline="0.25" toe_in_r="7" toe_in_l="0" width="0.4" height="0.05" length="0.05" image_width="1920" image_height="1080" image_format="MONO8" hfov="1.04" focus_near="0.3" r="0.1" g="0.1" b="0.1" />
 </robot>

File: i3dr_tools_ros_WS/src/i3dr_cameras/i3dr_stereo_camera-ros/urdf/i3dr_stereo_camera.urdf.xacro (robot description, xacro)
@@ -16,5 +16,5 @@
                 <origin xyz="0 0 0" rpy="0 0 0"/>
                 <geometry>
-                    <box size="${width} ${height} ${length}"/>
+                    <box size="${length} ${width} ${height}"/>
                 </geometry>
                 <material name="${camera_name}_camera_colour">
@@ -48,7 +48,7 @@
         </joint>
         <joint name="${camera_name}_depth_optical_joint" type="fixed">
-            <parent link="${camera_name}_cameraLeft_optical"/>
+            <parent link="${camera_name}_cameraRight"/>
             <child link="${camera_name}_depth_optical_frame"/>
-            <origin xyz="0 0 0" rpy="0 0 0" />
+            <origin xyz="0 0 0" rpy="${-pi/2} 0 ${(-pi/2)}" />
         </joint>
         <sensor name="${camera_name}_right_camera_sensor" update_rate="60">
@@ -62,9 +62,9 @@
             <parent link="${camera_name}_base_link"/>
             <child link="${camera_name}_center"/>
-            <origin xyz="${mount_offset_x} ${mount_offset_y} ${(length/2)+mount_offset_z}" rpy="0 0 ${-pi/2}" />
+            <origin xyz="${mount_offset_x} ${mount_offset_y} ${(height/2)+mount_offset_z}" rpy="0 0 ${-pi/2}" />
         </joint>
         <!-- Correct for IMU orientation, Z -> X -->
         <joint name="${camera_name}_imu_joint" type="fixed">
-            <origin xyz="0 0.015 -0.002" rpy="0 ${pi/2} 0" />
+            <origin xyz="0 0 0" rpy="0 ${pi/2} 0" />
             <parent link="${camera_name}_imu_link" />
             <child link="${camera_name}_base_link" />
