Commit message: add ur10 gui

File: i3dr_tools_ros_WS/src/i3dr_tools-ros/i3dr_cameras/i3dr_phobos_nuclear-ros/urdf/phobos_nuclear_scene.urdf.xacro (robot description, xacro)
@@ -9,4 +9,4 @@
     -->
     <xacro:include filename="$(find i3dr_phobos_nuclear)/urdf/phobos_nuclear.urdf.xacro"/>
-    <xacro:i3dr_phobos_nuclear camera_name="phobos_nuclear" en_mesh="false"/>
+    <xacro:i3dr_phobos_nuclear camera_name="phobos_nuclear" en_mesh="true"/>
 </robot>
